File: hardware/airguard_v1.sch (KiCad schematic (older format))
At the start: 2 parts, among them U1 MH-Z19B, U2 ESP32_DEVKIT_C

Commit message: Adding the OLED and all 3d models; connecting some of the signals to the corresponding ESP32 pins
Parts:
- added U3: SSD1306, footprints:SSD1306, symbol SSD1306-128x64_OLED:SSD1306
Connections:
- net +3V3: now also U3.2 (VCC)
- net GND: now also U3.1 (GND)
- net RXD2: now reaches U2.27 (IO16)
- net RXD2: now also U1.3 (TXD)
- net TXD2: now reaches U2.28 (IO17)
- net TXD2: now also U1.2 (RXD)
- net SDA: now reaches U2.33 (IO21)
- net SDA: now also U3.4 (SDA)
- net SCL: now reaches U2.36 (IO22)
- net SCL: now also U3.3 (SCL)
- net CAL: now reaches U1.5 (HD)
- no-connect marks 0 -> 2
Other:
- note added: "need to check if these displays have an onboard 3.3V regulator already"
- note added: "used for CP2102 UART"
Changed lines of the file:
@@
 	0    -1   -1   0
 $EndComp
+$Comp
+L SSD1306-128x64_OLED:SSD1306 U3
+U 1 1 615249EE
+P 2650 2300
+F 0 "U3" H 2928 2404 50  0000 L CNN
+F 1 "SSD1306" H 2928 2313 50  0000 L CNN
+F 2 "footprints:SSD1306" H 2650 2550 50  0001 C CNN
+F 3 "" H 2650 2550 50  0001 C CNN
+	1    2650 2300
+	1    0    0    -1
+$EndComp
+$Comp
+L power:+3.3V #PWR?
+U 1 1 615271EB
+P 2600 1950
+F 0 "#PWR?" H 2600 1800 50  0001 C CNN
+F 1 "+3.3V" H 2500 2400 50  0000 L CNN
+F 2 "" H 2600 1950 50  0001 C CNN
+F 3 "" H 2600 1950 50  0001 C CNN
+	1    2600 1950
+	1    0    0    -1
+$EndComp
+$Comp
+L power:GND #PWR?
+U 1 1 61527846
+P 2500 1950
+F 0 "#PWR?" H 2500 1700 50  0001 C CNN
+F 1 "GND" H 2500 1650 50  0000 C CNN
+F 2 "" H 2500 1950 50  0001 C CNN
+F 3 "" H 2500 1950 50  0001 C CNN
+	1    2500 1950
+	-1   0    0    1
+$EndComp
+Text GLabel 2700 1950 1    50   Input ~ 0
+SCL
+Text GLabel 2800 1950 1    50   Input ~ 0
+SDA
+Text GLabel 5700 2900 2    50   Input ~ 0
+SCL
+Text GLabel 5700 3200 2    50   Input ~ 0
+SDA
+NoConn ~ 5700 3000
+NoConn ~ 5700 3100
+Text Notes 5750 3050 0    50   ~ 0
+used for CP2102 UART
+Text GLabel 2300 3600 0    50   Input ~ 0
+RXD2
+Text GLabel 2300 3700 0    50   Input ~ 0
+TXD2
+Text GLabel 5700 3700 2    50   Input ~ 0
+TXD2
+Text GLabel 5700 3800 2    50   Input ~ 0
+RXD2
+Text Notes 1500 2750 0    50   ~ 0
+need to check if these displays have an onboard 3.3V regulator already
+Text GLabel 3200 3600 2    50   Input ~ 0
+CAL
+Text GLabel 3950 3500 2    50   Input ~ 0
+CAL
 $EndSCHEMATC
