File: hardware/main-pcb/airguard_v1.sch (KiCad schematic (older format))
At the start: 35 parts, among them J1 Conn_01x04_Female, J2 Conn_01x05_Female, J3 Conn_01x04_Female, J4 Conn_01x19_Female, J5 Conn_01x19_Female, J6 Conn_01x04_Female, Q1 PN2222A, Q2 PN2222A, Q3 PN2222A, Q4 PN2222A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

Commit message: updated main board to R3
Parts:
- added C1: CP, footprints:can-cap11x6.3, symbol Device:CP
- added X1: Badgelife_sao_connector_v169bis, badgelife_sao_v169bis:Badgelife-SAOv169-SAO-2x3, symbol badgelife_shitty_addon_v169bis:Badgelife_sao_connector_v169bis
- DZELTENS: renamed from DZELTENS1; footprint LEDs:LED_D10.0mm -> footprints:LED_D10.0mm
- J2: footprint (none) -> Oddities:Dummy_Empty
- R1, R10, R2, R3, R4, R6, R7, R8, R9: value R 4.7K -> 4700Ω
- R11, R12, R13: value 68R -> 68Ω
- R14, R15: value 33R -> 33Ω
- SARKANS: renamed from SARKANS1; footprint LEDs:LED_D10.0mm -> footprints:LED_D10.0mm
- ZAĻŠ: renamed from ZALS1; footprint LEDs:LED_D10.0mm -> footprints:LED_D10.0mm
Connections:
- net +3V3: now also X1.1 (VCC)
- net +5V: now also C1.1
- net GND: now also C1.2, X1.2 (GND)
- net SCL: now also X1.4 (SCL)
- net SDA: now also X1.3 (SDA)
- net SAO_GPIO2: now reaches U2.15 (IO13)
- net SAO_GPIO2: now also X1.6 (GPIO2)
- net SAO_GPIO1: now reaches U2.30 (IO18)
- net SAO_GPIO1: now also X1.5 (GPIO1)
Other:
- note added: "ACIS"
- note added: "BALSS"
- note added: "CO2 SENSORS"
- note added: "DZELTENĀ LED"
- note added: "EKRĀNS"
- note added: "GAISA SARGS R03"
- note added: "GAISMAS SENSORS"
- note added: "NEREDZAMĀS DETAĻAS"
- note added: "POGA"
- note added: "SAO \n(AKSESUĀRU CAURUMI)"
- note added: "SARKANĀ LED"
- note added: "SMADZENES"
- note added: "TIKAI DETAĻU SARAKSTAM"
- note added: "ZAĻĀ LED"
- note removed: "AMB LIGHT DETECT"
- note removed: "BEEP"
- note removed: "BUTTON"
- note removed: "CO2 SENSOR"
- note removed: "DUMMY PARTS"
- note removed: "ESP32 DEVKIT C"
- note removed: "EYES"
- note removed: "FOR BoM ONLY"
- note removed: "GAISA SARGS"
- note removed: "GREEN LED"
- note removed: "I2C OLED"
- note removed: "LCSC part \ndoesn't seem\nto specify polarity\nnot sure how to handle"
- note removed: "RED LED"
- note removed: "YELLOW LED"
- moved on the sheet: D1, D2, J1, J2, J3, J4, J5, J6, R1, R14, R15, R2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

Commit message: plot sch
Parts:
- renumbered DZELTENS to DZELTENS1, SARKANS to SARKANS1, ZAĻŠ to ZAĻŠ1
Other:
- note added: "GAISA SARGS R3"
- note removed: "GAISA SARGS R03"
Changed lines of the file:
@@
 $EndComp
 $Comp
-L Device:LED SARKANS
+L Device:LED SARKANS1
 U 1 1 6186E917
 P 10350 1350
-F 0 "SARKANS" V 10389 1232 50  0000 R CNN
+F 0 "SARKANS1" V 10389 1232 50  0000 R CNN
 F 1 "LED_RED" V 10298 1232 50  0000 R CNN
 F 2 "footprints:LED_D10.0mm" H 10350 1350 50  0001 C CNN
@@
 $EndComp
 $Comp
-L Device:LED DZELTENS
+L Device:LED DZELTENS1
 U 1 1 61890C9C
 P 10350 3200
-F 0 "DZELTENS" V 10389 3082 50  0000 R CNN
+F 0 "DZELTENS1" V 10389 3082 50  0000 R CNN
 F 1 "LED_YELLOW" V 10298 3082 50  0000 R CNN
 F 2 "footprints:LED_D10.0mm" H 10350 3200 50  0001 C CNN
@@
 $EndComp
 $Comp
-L Device:LED ZAĻŠ
+L Device:LED ZAĻŠ1
 U 1 1 61896192
 P 10350 5050
-F 0 "ZAĻŠ" V 10389 4932 50  0000 R CNN
+F 0 "ZAĻŠ1" V 10389 4932 50  0000 R CNN
 F 1 "LED_GREEN" V 10298 4932 50  0000 R CNN
 F 2 "footprints:LED_D10.0mm" H 10350 5050 50  0001 C CNN
@@
 	7150 6250 8900 6250
 Text Notes 750  1000 0    236  Italic 47
-GAISA SARGS R03
+GAISA SARGS R3
 $Comp
 L Switch:SW_Push SW1
