File: hardware/main-pcb/airguard_v1-aranet-logo.kicad_pcb (KiCad board)
At the start: 2 copper layers, 169.1 x 252.5 mm, 38 parts, among them J1 Conn_01x04_Female, J2 Conn_01x05_Female, J3 Conn_01x04_Female, J4 Conn_01x19_Female, J5 Conn_01x19_Female, J6 Conn_01x04_Female, Q1 PN2222A, Q2 PN2222A, Q3 PN2222A, Q4 PN2222A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

Commit message: added sponsor logos -mask only-
Parts:
- added Ref**: Val**, ziedotaju-logo:aranet-logo-mask-only, F.Cu at (146.5, 90.8)
